File: akami.sch (KiCad schematic (older format))
At the start: 49 parts, among them J1 USB_C_Receptacle_USB2.0, Q1 P MOSFET, Q2 P MOSFET, U1 nRF52840, U2 TP4054, U3 AP2112K-3.3, U4 ProMicro_2, Y1 32MHz, Y2 32.768 kHz

Commit message: more stuff
Parts:
- added J2, J3: Conn_01x01, footprints:1pin_conn, symbol Connector_Generic:Conn_01x01
- added TP3: TestPoint, TestPoint:TestPoint_Pad_1.0x1.0mm, symbol Connector:TestPoint
- added TP4: TestPoint, footprints:circular-pad-0.3mm, symbol Connector:TestPoint
- C17, C18: value 12pF -> 3.3pF; LCSC Part C1547 -> C1565
- C6, C7: value 12pF -> 10pF; LCSC Part C1547 -> C32949
Connections:
- net GND: now also J3.1 (Pin_1)
- net VBAT: now also J2.1 (Pin_1)
- net VDD_NRF: now also TP3.1
- net ANTENNA: now reaches C22.2, C5.2, L1.1
- net ANTENNA: now also TP4.1
- no-connect marks 24 -> 23
Other:
- note added: "3V3_OUT Control"
- note added: "Battery Charger"
- note added: "Battery Voltage Divider"
- note added: "Decoupling Capacitors"
- note added: "Power"
- note added: "Pro Micro Footprint"
- note added: "Status LED"
- note added: "USB Connector"
- note added: "https://devzone.nordicsemi.com/nordic/nordic-blog\n/b/blog/posts/measuring-lithium-battery-voltage-with-nrf52"
- note added: "nobody makes 4M resistors\nand 0402 2M resistors are extended\nso, use a 3M 0603 and\na 1M 0402 (both basic) in series"
- note added: "this is so the antenna trace\ndoesn't get removed"
- note removed: "ANTENNA"
- note removed: "https://devzone.nordicsemi.com/nordic/nordic-blog/b/blog/posts/measuring-lithium-battery-voltage-with-nrf52"
- note removed: "nobody makes 4M resistors, and 0402 2M resistors are extended\nso, use a 3M 0603 and a 1M 0402 (both basic) in series"
- moved on the sheet: C1, C19, C2, C20, C21, C3, C4, C8, D1, D2, D3, J1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

Commit message: stuff
Parts:
- added NT1: Net-Tie_2, footprints:net-tie-2-tiny, symbol Device:Net-Tie_2
- C12: value 820pF -> 1nF; LCSC Part C307452 -> C1523
- C17, C18: value 3.3pF -> 15pF; LCSC Part C1565 -> C1548
- Q1, Q2: value P MOSFET -> AO3401A; LCSC Part C10487 -> C15127
- Y1: LCSC Part C383840 -> C254298
- Y2: footprint Crystal:Crystal_SMD_2012-2Pin_2.0x1.2mm -> Crystal:Crystal_SMD_3215-2Pin_3.2x1.5mm; LCSC Part C99009 -> C32346
Connections:
- net GND: now also NT1.2
- net VSS_PA: now also NT1.1
Other:
- note added: "https://devzone.nordicsemi.com/f/nordic-q-a\n/37758/dec5-decoupling-capacitor-value\n\n=> C12 can be 1nF"
- moved on the sheet: C20, L2, L3
